Commit message: Added gearboxes

File: soft_hand_description/model/soft_hand.urdf.xacro (robot description, xacro)
@@ -134,4 +134,18 @@
 			</collision>
 		</link>
+		<gazebo>
+			<joint name="${name}_inner_joint_gearbox" type="gearbox">
+			<parent>${name}_knuckle_link</parent>
+			<child>${name}_proximal_link</child>
+			<gearbox_ratio>-1.0</gearbox_ratio>
+			<gearbox_reference_body>${name}_fake_link1</gearbox_reference_body>
+			<axis>
+				<xyz>0.0 -1.0 0.0</xyz>
+			</axis>
+			<axis2>
+				<xyz>0.0 -1.0 0.0</xyz>
+			</axis2>
+			</joint>
+		</gazebo>
 		<!-- MIDDLE PHALANGE -->
 		<joint name="${name}_middle_joint" type="revolute">
@@ -178,4 +192,18 @@
 			</collision>
 		</link>
+		<gazebo>
+			<joint name="${name}_middle_joint_gearbox" type="gearbox">
+			<parent>${name}_proximal_link</parent>
+			<child>${name}_middle_link</child>
+			<gearbox_ratio>-1.0</gearbox_ratio>
+			<gearbox_reference_body>${name}_fake_link2</gearbox_reference_body>
+			<axis>
+				<xyz>0.0 -1.0 0.0</xyz>
+			</axis>
+			<axis2>
+				<xyz>0.0 -1.0 0.0</xyz>
+			</axis2>
+			</joint>
+		</gazebo>
 		<!-- DISTAL PHALANGE -->
 		<joint name="${name}_outer_joint" type="revolute">
@@ -222,4 +250,18 @@
 			</collision>
 		</link>
+		<gazebo>
+			<joint name="${name}_outer_joint_gearbox" type="gearbox">
+			<parent>${name}_middle_link</parent>
+			<child>${name}_distal_link</child>
+			<gearbox_ratio>-1.0</gearbox_ratio>
+			<gearbox_reference_body>${name}_fake_link3</gearbox_reference_body>
+			<axis>
+				<xyz>0.0 -1.0 0.0</xyz>
+			</axis>
+			<axis2>
+				<xyz>0.0 -1.0 0.0</xyz>
+			</axis2>
+			</joint>
+		</gazebo>
 	</xacro:macro>
 	<!-- THUMB MODEL -->
@@ -343,4 +385,18 @@
 			</collision>
 		</link>
+		<gazebo>
+			<joint name="${name}_inner_joint_gearbox" type="gearbox">
+			<parent>${name}_knuckle_link</parent>
+			<child>${name}_proximal_link</child>
+			<gearbox_ratio>-1.0</gearbox_ratio>
+			<gearbox_reference_body>${name}_fake_link1</gearbox_reference_body>
+			<axis>
+				<xyz>0.0 -1.0 0.0</xyz>
+			</axis>
+			<axis2>
+				<xyz>0.0 -1.0 0.0</xyz>
+			</axis2>
+			</joint>
+		</gazebo>
 		<!-- DISTAL PHALANGE -->
 		<joint name="${name}_outer_joint" type="revolute">
@@ -387,4 +443,18 @@
 			</collision>
 		</link>
+		<gazebo>
+			<joint name="${name}_outer_joint_gearbox" type="gearbox">
+			<parent>${name}_proximal_link</parent>
+			<child>${name}_distal_link</child>
+			<gearbox_ratio>-1.0</gearbox_ratio>
+			<gearbox_reference_body>${name}_fake_link3</gearbox_reference_body>
+			<axis>
+				<xyz>0.0 -1.0 0.0</xyz>
+			</axis>
+			<axis2>
+				<xyz>0.0 -1.0 0.0</xyz>
+			</axis2>
+			</joint>
+		</gazebo>
 	</xacro:macro>
 	<!-- SOFT HAND MODEL -->
